File: SDRReciever/_autosave-SDRReciever.sch (KiCad schematic (older format))
At the start: 80 parts, among them J1 Conn_Coaxial, J10 I_0, J11 I_180, J12 Q_90, J13 Q_270, J14 I_OUT, J15 Q_OUT, J16 5V, J17 4.3V, J18 Conn_01x02_Female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

Commit message: Organized images and added schematic images
Other:
- note added: "Toroid Info:\nT37-6: 3nH per turns^2\nT50-6: 4nH per turns^2\nSee datasheet for more info"
Changed lines of the file:
@@
 Wire Notes Line
 	4150 1850 4150 1700
+Text Notes 625  925  0    50   ~ 0
+Toroid Info:\nT37-6: 3nH per turns^2\nT50-6: 4nH per turns^2\nSee datasheet for more info
+Wire Notes Line
+	600  600  600  950
+Wire Notes Line
+	600  950  1750 950
+Wire Notes Line
+	1750 950  1750 600
+Wire Notes Line
+	1750 600  600  600
 $EndSCHEMATC
