File: SDRReceiver_Rev2/SDRReciever/SDRReciever.sch (KiCad schematic (older format))
At the start: 78 parts, among them J1 Conn_Coaxial, J10 I_0, J11 I_180, J12 Q_90, J13 Q_270, J14 I_OUT, J15 Q_OUT, J16 5V, J17 4.3V, J18 Conn_01x02_Female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

Commit message: Fixed the Rev2 schematic from being pulled apart for screenshots
Parts:
- added RV1: 100k, symbol Device:R_POT
- added U7: LM741, symbol Amplifier_Operational:LM741
- C1: value 220pF -> 620pF
- C2: value 1nF -> 910pF
- C3: value 220pF -> 150pF
- J5: value CLK_2 -> CLK_1
- J6: value CLK_3 -> CLK_2
- J7: value CLK_1 -> CLK_0
- L1: value 1.3uH -> 820nH
- L2: value 200nH -> 560nH
- L3: value 1.3uH -> 3.6uH
- R3, R4: value 33 -> 1k
- R7, R8: value 10k -> 1k; footprint Resistor_THT:R_Axial_DIN0207_L6.3mm_D2.5mm_P7.62mm_Horizontal -> (none)
- Y1: value Crystal -> ATS250
Connections:
- wire segments 235 -> 249
- no-connect marks 25 -> 27
Other:
- note added: "00 = 0°"
- note added: "01 = 90°"
- note added: "10 = 180°"
- note added: "11 = 270°"
- note added: "Bandpass Filter 5-18MHz (3rd Order, Series-First Bessel)\nBy doing Series-First, DC signals cannot pass through the capacitor (C2), \nallowing better control over the DC offset going into the op-amps"
- note added: "Full Scale Input \nSignal Level Typ: 1.0 Vrms\nInput R = 55kΩ."
- note added: "I Signal"
- note added: "Johnson Counter CLK/4 Circuit\nusing 74AC74 dual flip flops"
- note added: "Jumper for\npreventing \nground loops"
- note added: "Low Noise Instrumentation Amplifiers\nGain Controlled by 1 Resistor. J18 and \nJ19 used for testing for desired gain"
- note added: "Pull-Up Resistors for I2C lines see the \nSi5351 datasheet for details"
- note added: "Q Signal"
- note added: "SDA and SCL are I2C Control Signals \nfor the Si5351 Clock Generator"
- note added: "T37-6 Toroid:\n17 turns"
- note added: "T50-6 Toroid: \n12 turns"
- note added: "T50-6 Toroid: \n30 turns"
- note added: "The ATS250 is \na low-cost 25 \nMHz crystal"
- note added: "The INA821ID Amps require the REF\ninput to have a voltage source with a\nlow output impedence. The LM741\nvoltage buffer handles this"
- note added: "The dual op amp symbol was made\nby me. It is not implying that the V+ of one\nis connected to the V- of the other, but that they\nshare the same power and ground pins"
- note added: "Toroid Info:\nT37-6: 3nH per turns^2\nT50-6: 4nH per turns^2\nSee datasheet for more info"
- note added: "Tunable\n2.15V Bias"
- note added: "Two-Pole Low Pass Filter\nUsing 2-Channel Op Amp\n100kHz Cutoff, no gain"
- note added: "Voltage Protection Diodes:\nThese will prevent too large of signals \nfrom coming through"
- note added: "Voltage Smoother \nFor PC 5V power to \neliminate supply noise"
- note added: "With 5-10MHz, \nCLK_0 will \nbe around \n20 - 40 MHz"
- note removed: "0 deg"
- note removed: "180 deg"
- note removed: "2.15V Bias"
- note removed: "270 deg"
- note removed: "90 deg"
- note removed: "Bandpass Filter 5-18MHz\n(3rd Order, Series-First Bessel)"
- note removed: "Full Scale Input \nSignal Level Typ: 1.0 Vrms\n\nInput R = 55 kOhm"
- note removed: "I Sig. From Inst. Amps"
- note removed: "I2C Lines to Clock Generator"
- note removed: "I2C Lines\nfrom Arduino \n(A4 and A5)"
- note removed: "Jumper to prevent \nground loops"
- note removed: "Local Oscilator lines\nfrom Johnson Counter"
- note removed: "Low Noise Instrumentation Amplifiers\nGain Controlled by 1 Resistor"
- note removed: "Q Sig. From Inst. Amps"
- note removed: "Select Line\nto Tayloe \nMixer MUX"
- note removed: "Signal from \nBandpass Filter"
- note removed: "Signal in \nfrom Antenna"
- note removed: "Signal to \nTayloe Mixer"
- note removed: "T37-6 Toroid: \n8 turns"
- note removed: "T50-6 Toroid:\n18 turns"
- note removed: "To DC Offset"
- note removed: "To Lowpass Filter"
- note removed: "Two-Pole Low Pass Filter\nUsing 2-Channel Op Amp"
- note removed: "Voltage Protection \n Diodes"
- note removed: "Voltage Smoother For\nPC 5V power"
- note removed: "With 5-10MHz, LO will be\naround 20 - 40 MHz"
- moved on the sheet: A1, C1, C10, C11, C12, C13, C14, C15, C16, C17, C18, C19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
